Commit message: add phosphobot support

File: om6dof_bringup/urdf/om6dof.ros2_control.xacro (robot description, xacro)
@@ -19,4 +19,5 @@
       port_name:=/dev/ttyUSB0
       baudrate:=1000000
+      consecutive_failure_shutdown_threshold:=10
       use_fake_hardware:=false">
     <ros2_control name="${name}" type="system">
@@ -33,4 +34,5 @@
           <param name="baud_rate">${baudrate}</param>
           <param name="error_timeout_ms">500</param>
+          <param name="consecutive_failure_shutdown_threshold">${consecutive_failure_shutdown_threshold}</param>
           <!-- Plain SyncRead from the start. FastSyncRead is tighter on bus
                timing and throws -3001 SYNC_READ_FAIL on the first cycle after

File: om6dof_bringup/urdf/om6dof.urdf.xacro (robot description, xacro)
@@ -4,4 +4,7 @@
   <xacro:arg name="baud_rate" default="1000000"/>
   <xacro:arg name="use_fake_hardware" default="false"/>
+  <!-- Runtime communication fail-safe settings are kept in one editable file. -->
+  <xacro:property name="hardware_safety"
+    value="${xacro.load_yaml('$(find om6dof_bringup)/config/hardware_safety.yaml')}"/>
   <xacro:include filename="$(find om6dof_description)/urdf/om6dof.urdf.xacro"/>
   <xacro:include filename="$(find om6dof_bringup)/urdf/om6dof.ros2_control.xacro"/>
@@ -10,4 +13,5 @@
     port_name="$(arg port_name)"
     baudrate="$(arg baud_rate)"
+    consecutive_failure_shutdown_threshold="${hardware_safety['consecutive_failure_shutdown_threshold']}"
     use_fake_hardware="$(arg use_fake_hardware)"/>
 </robot>
