Commit message: add gravity compensation

File: om6dof_bringup/urdf/om6dof.ros2_control.current.xacro (robot description, xacro)
@@ -1,19 +1,14 @@
 <?xml version="1.0"?>
 <!--
-  Current-limited variant of om6dof.ros2_control.xacro, for leading the arm
-  by hand.
+  Effort-command variant of om6dof.ros2_control.xacro.
   WHAT DIFFERS FROM THE STANDARD FILE
     each arm joint gains an "effort" command interface
     each servo gains a "Goal Current" command interface
-    Operating Mode goes from 3 (position) to 5 (current-based position)
-  WHY MODE 5 AND NOT MODE 0
-    Mode 0 is pure current control. The servo stops holding position at all,
-    so if the compensation model is wrong, or the node stops, the arm falls
-    under its own weight. Mode 5 keeps the position loop and caps how hard it
-    may pull: command a small Goal Current and the arm becomes backdrivable,
-    light enough to lead by hand, while still holding its pose when let go.
-    The gripper on this arm already runs in mode 5.
-    Mode 0 is the endpoint once the model is trusted at every pose, including
-    standing still. That is not yet true, so it is not this file.
+    Operating mode for arm joints is selected by arm_operating_mode:
+    5 = current-based position; 0 = signed, pure current control.
+  MODE 0 WARNING
+    In pure current control the position loop is absent. It is suitable only
+    with a live, signed gravity-compensation controller and a supported arm.
+    The gripper always remains in mode 5.
   NOT LOADED BY DEFAULT
     The standard bringup keeps using om6dof.ros2_control.xacro. Loading this
@@ -41,5 +36,6 @@
       baudrate:=1000000
       consecutive_failure_shutdown_threshold:=10
-      use_fake_hardware:=false">
+      use_fake_hardware:=false
+      arm_operating_mode:=5">
     <ros2_control name="${name}" type="system">
       <xacro:if value="${use_fake_hardware}">
@@ -172,12 +168,18 @@
         <param name="type">dxl</param>
         <param name="ID">31</param>
-        <command_interface name="Goal Position"/>
-        <command_interface name="Goal Current"/>
-        <state_interface name="Present Position"/>
-        <state_interface name="Present Velocity"/>
-        <state_interface name="Present Current"/>
-        <state_interface name="Torque Enable"/>
-        <state_interface name="Present Input Voltage"/>
-        <param name="Operating Mode">5</param>
+        <param name="Bus Watchdog">10</param>
+        <command_interface name="Goal Position"/>
+        <command_interface name="Goal Current"/>
+        <state_interface name="Present Position"/>
+        <state_interface name="Present Velocity"/>
+        <state_interface name="Present Current"/>
+        <state_interface name="Torque Enable"/>
+        <state_interface name="Present Input Voltage"/>
+        <param name="Operating Mode">${arm_operating_mode}</param>
+        <!-- Mode 0 is accepted by the hardware driver only after an explicit
+             zero-current packet, preventing torque enable with a stale value. -->
+        <xacro:if value="${int(arm_operating_mode) == 0}">
+          <param name="Goal Current">0</param>
+        </xacro:if>
         <param name="Position P Gain">800</param>
         <param name="Position I Gain">100</param>
@@ -191,12 +193,16 @@
         <param name="type">dxl</param>
         <param name="ID">32</param>
-        <command_interface name="Goal Position"/>
-        <command_interface name="Goal Current"/>
-        <state_interface name="Present Position"/>
-        <state_interface name="Present Velocity"/>
-        <state_interface name="Present Current"/>
-        <state_interface name="Torque Enable"/>
-        <state_interface name="Present Input Voltage"/>
-        <param name="Operating Mode">5</param>
+        <param name="Bus Watchdog">10</param>
+        <command_interface name="Goal Position"/>
+        <command_interface name="Goal Current"/>
+        <state_interface name="Present Position"/>
+        <state_interface name="Present Velocity"/>
+        <state_interface name="Present Current"/>
+        <state_interface name="Torque Enable"/>
+        <state_interface name="Present Input Voltage"/>
+        <param name="Operating Mode">${arm_operating_mode}</param>
+        <xacro:if value="${int(arm_operating_mode) == 0}">
+          <param name="Goal Current">0</param>
+        </xacro:if>
         <param name="Position P Gain">800</param>
         <param name="Position I Gain">100</param>
@@ -210,12 +216,16 @@
         <param name="type">dxl</param>
         <param name="ID">33</param>
-        <command_interface name="Goal Position"/>
-        <command_interface name="Goal Current"/>
-        <state_interface name="Present Position"/>
-        <state_interface name="Present Velocity"/>
-        <state_interface name="Present Current"/>
-        <state_interface name="Torque Enable"/>
-        <state_interface name="Present Input Voltage"/>
-        <param name="Operating Mode">5</param>
+        <param name="Bus Watchdog">10</param>
+        <command_interface name="Goal Position"/>
+        <command_interface name="Goal Current"/>
+        <state_interface name="Present Position"/>
+        <state_interface name="Present Velocity"/>
+        <state_interface name="Present Current"/>
+        <state_interface name="Torque Enable"/>
+        <state_interface name="Present Input Voltage"/>
+        <param name="Operating Mode">${arm_operating_mode}</param>
+        <xacro:if value="${int(arm_operating_mode) == 0}">
+          <param name="Goal Current">0</param>
+        </xacro:if>
         <param name="Position P Gain">800</param>
         <param name="Position I Gain">100</param>
@@ -229,12 +239,16 @@
         <param name="type">dxl</param>
         <param name="ID">24</param>
-        <command_interface name="Goal Position"/>
-        <command_interface name="Goal Current"/>
-        <state_interface name="Present Position"/>
-        <state_interface name="Present Velocity"/>
-        <state_interface name="Present Current"/>
-        <state_interface name="Torque Enable"/>
-        <state_interface name="Present Input Voltage"/>
-        <param name="Operating Mode">5</param>
+        <param name="Bus Watchdog">10</param>
+        <command_interface name="Goal Position"/>
+        <command_interface name="Goal Current"/>
+        <state_interface name="Present Position"/>
+        <state_interface name="Present Velocity"/>
+        <state_interface name="Present Current"/>
+        <state_interface name="Torque Enable"/>
+        <state_interface name="Present Input Voltage"/>
+        <param name="Operating Mode">${arm_operating_mode}</param>
+        <xacro:if value="${int(arm_operating_mode) == 0}">
+          <param name="Goal Current">0</param>
+        </xacro:if>
         <param name="Position P Gain">800</param>
         <param name="Position I Gain">100</param>
@@ -248,12 +262,16 @@
         <param name="type">dxl</param>
         <param name="ID">35</param>
-        <command_interface name="Goal Position"/>
-        <command_interface name="Goal Current"/>
-        <state_interface name="Present Position"/>
-        <state_interface name="Present Velocity"/>
-        <state_interface name="Present Current"/>
-        <state_interface name="Torque Enable"/>
-        <state_interface name="Present Input Voltage"/>
-        <param name="Operating Mode">5</param>
+        <param name="Bus Watchdog">10</param>
+        <command_interface name="Goal Position"/>
+        <command_interface name="Goal Current"/>
+        <state_interface name="Present Position"/>
+        <state_interface name="Present Velocity"/>
+        <state_interface name="Present Current"/>
+        <state_interface name="Torque Enable"/>
+        <state_interface name="Present Input Voltage"/>
+        <param name="Operating Mode">${arm_operating_mode}</param>
+        <xacro:if value="${int(arm_operating_mode) == 0}">
+          <param name="Goal Current">0</param>
+        </xacro:if>
         <param name="Position P Gain">800</param>
         <param name="Position I Gain">100</param>
@@ -267,12 +285,16 @@
         <param name="type">dxl</param>
         <param name="ID">26</param>
-        <command_interface name="Goal Position"/>
-        <command_interface name="Goal Current"/>
-        <state_interface name="Present Position"/>
-        <state_interface name="Present Velocity"/>
-        <state_interface name="Present Current"/>
-        <state_interface name="Torque Enable"/>
-        <state_interface name="Present Input Voltage"/>
-        <param name="Operating Mode">5</param>
+        <param name="Bus Watchdog">10</param>
+        <command_interface name="Goal Position"/>
+        <command_interface name="Goal Current"/>
+        <state_interface name="Present Position"/>
+        <state_interface name="Present Velocity"/>
+        <state_interface name="Present Current"/>
+        <state_interface name="Torque Enable"/>
+        <state_interface name="Present Input Voltage"/>
+        <param name="Operating Mode">${arm_operating_mode}</param>
+        <xacro:if value="${int(arm_operating_mode) == 0}">
+          <param name="Goal Current">0</param>
+        </xacro:if>
         <param name="Position P Gain">800</param>
         <param name="Position I Gain">100</param>

File: om6dof_bringup/urdf/om6dof.ros2_control.xacro (robot description, xacro)
@@ -20,5 +20,6 @@
       baudrate:=1000000
       consecutive_failure_shutdown_threshold:=10
-      use_fake_hardware:=false">
+      use_fake_hardware:=false
+      arm_operating_mode:=5">
     <ros2_control name="${name}" type="system">
       <xacro:if value="${use_fake_hardware}">
@@ -145,4 +146,5 @@
         <param name="type">dxl</param>
         <param name="ID">31</param>
+        <param name="Bus Watchdog">10</param>
         <command_interface name="Goal Position"/>
         <state_interface name="Present Position"/>
@@ -163,4 +165,5 @@
         <param name="type">dxl</param>
         <param name="ID">32</param>
+        <param name="Bus Watchdog">10</param>
         <command_interface name="Goal Position"/>
         <state_interface name="Present Position"/>
@@ -181,4 +184,5 @@
         <param name="type">dxl</param>
         <param name="ID">33</param>
+        <param name="Bus Watchdog">10</param>
         <command_interface name="Goal Position"/>
         <state_interface name="Present Position"/>
@@ -199,4 +203,5 @@
         <param name="type">dxl</param>
         <param name="ID">24</param>
+        <param name="Bus Watchdog">10</param>
         <command_interface name="Goal Position"/>
         <state_interface name="Present Position"/>
@@ -217,4 +222,5 @@
         <param name="type">dxl</param>
         <param name="ID">35</param>
+        <param name="Bus Watchdog">10</param>
         <command_interface name="Goal Position"/>
         <state_interface name="Present Position"/>
@@ -235,4 +241,5 @@
         <param name="type">dxl</param>
         <param name="ID">26</param>
+        <param name="Bus Watchdog">10</param>
         <command_interface name="Goal Position"/>
         <state_interface name="Present Position"/>

File: om6dof_bringup/urdf/om6dof.urdf.xacro (robot description, xacro)
@@ -9,4 +9,7 @@
        becomes softer the moment it is loaded, so switch it deliberately. -->
   <xacro:arg name="current_control" default="false"/>
+  <!-- Passed through only when current_control is true.  5 retains the
+       Dynamixel position loop; 0 makes Goal Current a signed torque command. -->
+  <xacro:arg name="arm_operating_mode" default="5"/>
   <!-- Runtime communication fail-safe settings are kept in one editable file. -->
   <xacro:property name="hardware_safety"
@@ -26,4 +29,5 @@
     baudrate="$(arg baud_rate)"
     consecutive_failure_shutdown_threshold="${hardware_safety['consecutive_failure_shutdown_threshold']}"
-    use_fake_hardware="$(arg use_fake_hardware)"/>
+    use_fake_hardware="$(arg use_fake_hardware)"
+    arm_operating_mode="$(arg arm_operating_mode)"/>
 </robot>

File: om6dof_description/urdf/om6dof.urdf.xacro (robot description, xacro)
@@ -37,5 +37,5 @@
     </inertial>-->
      <inertial>
-      <origin xyz="3.0876154e-04 0.0000000e+00 -1.2176461e-04" />
+      <origin xyz="3.0876154e-04 0.00 0.018" />
       <mass value="7.9119962e-02" />
       <inertia ixx="1.2505234e-05" ixy="0.0" ixz="-1.7855208e-07"
@@ -497,4 +497,13 @@
       <material name="white"/>
     </visual>
+    <!-- Exact final-path validation uses the same fused bracket+D405 mesh.
+         The fast online reachability filter still uses conservative capsules,
+         so this triangle mesh is evaluated only for shortlisted paths. -->
+    <collision>
+      <origin xyz="0.0191 -0.0272 -0.0755" rpy="0 0 0"/>
+      <geometry>
+        <mesh filename="package://om6dof_description/meshes/d405_wrist_cam.stl" scale="0.001 0.001 0.001"/>
+      </geometry>
+    </collision>
     <xacro:if value="${payload_mass > 0.0}">
       <!-- Solid sphere: valid for any mass, and gravity reads none of it. -->
@@ -558,14 +567,14 @@
        symmetric in it; unlike the bracket rotation there is no photo of the assembled camera
        to check against). That 9 mm is left off (optical frame kept on the centerline) rather
-       than guessing its sign: it only shifts the drawn TF pose in RViz, never the
-       reconstructed point cloud, because the perception node deprojects with librealsense's
-       own live intrinsics (fx, fy, ppx, ppy read from the camera at runtime), not this static
-       offset.
-       d405_depth_optical_frame's rotation relative to d405_link is left as identity: baseline
-       (d405.stl local X) lands within 0.012 deg of link7's own +Y axis, and forward (local Z)
-       within 25 deg of link7's +Z, exactly what X-right/Y-down/Z-forward should look like if
-       d405.stl's mesh axes were already authored in that convention, which is plausible for a
-       mesh sourced for URDF/ROS use. Like the 9 mm above, this is not verified against the
-       real hardware's markings.
+       than guessing its sign. This leaves an unknown rigid translation of up to 9 mm in the
+       reconstructed world-frame cloud: live intrinsics determine the deprojected ray, but do
+       not replace the housing-to-imager extrinsic translation.
+       d405.stl local +Z is camera-forward, but its local +X and +Y are image-left and image-up.
+       This was cross-checked against google-deepmind/mujoco_menagerie's ALOHA model, which
+       places the D405 mesh and wrist camera in the same parent frame, and against the local
+       mesh geometry (the local file is a decimated copy with the same axes). ROS optical is
+       X-right/Y-down/Z-forward, so d405_depth_optical_frame needs a pi roll about local +Z:
+       diag(-1,-1,+1). This preserves the verified forward direction (25 deg from link7 +Z)
+       while correcting both image-plane axis signs.
   -->
   <joint name="d405_link_joint" type="fixed">
@@ -578,5 +587,5 @@
     <!-- -0.0037 m: Table 4-16 "Depth Start Point" for D405, 3.7 mm behind the front cover
          glass (local -Z, back toward the sensor); see the derivation above. -->
-    <origin xyz="0 0 -0.0037" rpy="0 0 0"/>
+    <origin xyz="0 0 -0.0037" rpy="0 0 ${pi}"/>
     <parent link="d405_link"/>
     <child link="d405_depth_optical_frame"/>
