Commit message: add gemini based object detection

File: om6dof_bringup/urdf/om6dof.ros2_control.current.xacro (robot description, xacro)
@@ -36,6 +36,9 @@
       baudrate:=1000000
       consecutive_failure_shutdown_threshold:=10
+      read_packet_timeout_ms:=30.0
+      read_transport_mode:=multi_sync
       use_fake_hardware:=false
-      arm_operating_mode:=5">
+      arm_operating_mode:=5
+      torque_off_diagnostic_mode:=false">
     <ros2_control name="${name}" type="system">
       <xacro:if value="${use_fake_hardware}">
@@ -52,4 +55,7 @@
           <param name="error_timeout_ms">500</param>
           <param name="consecutive_failure_shutdown_threshold">${consecutive_failure_shutdown_threshold}</param>
+          <param name="read_packet_timeout_ms">${read_packet_timeout_ms}</param>
+          <param name="read_transport_mode">${read_transport_mode}</param>
+          <param name="torque_off_diagnostic_mode">${torque_off_diagnostic_mode}</param>
           <!-- Plain SyncRead from the start. FastSyncRead is tighter on bus
                timing and throws -3001 SYNC_READ_FAIL on the first cycle after
@@ -176,4 +182,5 @@
         <state_interface name="Torque Enable"/>
         <state_interface name="Present Input Voltage"/>
+        <state_interface name="Hardware Error Status"/>
         <param name="Operating Mode">${arm_operating_mode}</param>
         <!-- Mode 0 is accepted by the hardware driver only after an explicit
@@ -201,4 +208,5 @@
         <state_interface name="Torque Enable"/>
         <state_interface name="Present Input Voltage"/>
+        <state_interface name="Hardware Error Status"/>
         <param name="Operating Mode">${arm_operating_mode}</param>
         <xacro:if value="${int(arm_operating_mode) == 0}">
@@ -224,4 +232,5 @@
         <state_interface name="Torque Enable"/>
         <state_interface name="Present Input Voltage"/>
+        <state_interface name="Hardware Error Status"/>
         <param name="Operating Mode">${arm_operating_mode}</param>
         <xacro:if value="${int(arm_operating_mode) == 0}">
@@ -247,4 +256,5 @@
         <state_interface name="Torque Enable"/>
         <state_interface name="Present Input Voltage"/>
+        <state_interface name="Hardware Error Status"/>
         <param name="Operating Mode">${arm_operating_mode}</param>
         <xacro:if value="${int(arm_operating_mode) == 0}">
@@ -270,4 +280,5 @@
         <state_interface name="Torque Enable"/>
         <state_interface name="Present Input Voltage"/>
+        <state_interface name="Hardware Error Status"/>
         <param name="Operating Mode">${arm_operating_mode}</param>
         <xacro:if value="${int(arm_operating_mode) == 0}">
@@ -293,4 +304,5 @@
         <state_interface name="Torque Enable"/>
         <state_interface name="Present Input Voltage"/>
+        <state_interface name="Hardware Error Status"/>
         <param name="Operating Mode">${arm_operating_mode}</param>
         <xacro:if value="${int(arm_operating_mode) == 0}">
@@ -316,4 +328,5 @@
         <state_interface name="Torque Enable"/>
         <state_interface name="Present Input Voltage"/>
+        <state_interface name="Hardware Error Status"/>
         <param name="Operating Mode">5</param>
         <param name="Profile Velocity">20</param>

File: om6dof_bringup/urdf/om6dof.ros2_control.xacro (robot description, xacro)
@@ -20,6 +20,9 @@
       baudrate:=1000000
       consecutive_failure_shutdown_threshold:=10
+      read_packet_timeout_ms:=30.0
+      read_transport_mode:=multi_sync
       use_fake_hardware:=false
-      arm_operating_mode:=5">
+      arm_operating_mode:=5
+      torque_off_diagnostic_mode:=false">
     <ros2_control name="${name}" type="system">
       <xacro:if value="${use_fake_hardware}">
@@ -36,4 +39,7 @@
           <param name="error_timeout_ms">500</param>
           <param name="consecutive_failure_shutdown_threshold">${consecutive_failure_shutdown_threshold}</param>
+          <param name="read_packet_timeout_ms">${read_packet_timeout_ms}</param>
+          <param name="read_transport_mode">${read_transport_mode}</param>
+          <param name="torque_off_diagnostic_mode">${torque_off_diagnostic_mode}</param>
           <!-- Plain SyncRead from the start. FastSyncRead is tighter on bus
                timing and throws -3001 SYNC_READ_FAIL on the first cycle after
@@ -153,4 +159,5 @@
         <state_interface name="Torque Enable"/>
         <state_interface name="Present Input Voltage"/>
+        <state_interface name="Hardware Error Status"/>
         <param name="Operating Mode">3</param>
         <param name="Position P Gain">800</param>
@@ -172,4 +179,5 @@
         <state_interface name="Torque Enable"/>
         <state_interface name="Present Input Voltage"/>
+        <state_interface name="Hardware Error Status"/>
         <param name="Operating Mode">3</param>
         <param name="Position P Gain">800</param>
@@ -191,4 +199,5 @@
         <state_interface name="Torque Enable"/>
         <state_interface name="Present Input Voltage"/>
+        <state_interface name="Hardware Error Status"/>
         <param name="Operating Mode">3</param>
         <param name="Position P Gain">800</param>
@@ -210,4 +219,5 @@
         <state_interface name="Torque Enable"/>
         <state_interface name="Present Input Voltage"/>
+        <state_interface name="Hardware Error Status"/>
         <param name="Operating Mode">3</param>
         <param name="Position P Gain">800</param>
@@ -229,4 +239,5 @@
         <state_interface name="Torque Enable"/>
         <state_interface name="Present Input Voltage"/>
+        <state_interface name="Hardware Error Status"/>
         <param name="Operating Mode">3</param>
         <param name="Position P Gain">800</param>
@@ -248,4 +259,5 @@
         <state_interface name="Torque Enable"/>
         <state_interface name="Present Input Voltage"/>
+        <state_interface name="Hardware Error Status"/>
         <param name="Operating Mode">3</param>
         <param name="Position P Gain">800</param>
@@ -267,4 +279,5 @@
         <state_interface name="Torque Enable"/>
         <state_interface name="Present Input Voltage"/>
+        <state_interface name="Hardware Error Status"/>
         <param name="Operating Mode">5</param>
         <param name="Profile Velocity">20</param>

File: om6dof_bringup/urdf/om6dof.urdf.xacro (robot description, xacro)
@@ -12,4 +12,8 @@
        Dynamixel position loop; 0 makes Goal Current a signed torque command. -->
   <xacro:arg name="arm_operating_mode" default="5"/>
+  <!-- Internal fail-closed profile used only by torque_off_diagnostic.launch.py.
+       The driver treats this as an invariant: it forces torque off and rejects
+       every ROS path that could turn it back on. -->
+  <xacro:arg name="torque_off_diagnostic_mode" default="false"/>
   <!-- Runtime communication fail-safe settings are kept in one editable file. -->
   <xacro:property name="hardware_safety"
@@ -29,5 +33,8 @@
     baudrate="$(arg baud_rate)"
     consecutive_failure_shutdown_threshold="${hardware_safety['consecutive_failure_shutdown_threshold']}"
+    read_packet_timeout_ms="${hardware_safety['read_packet_timeout_ms']}"
+    read_transport_mode="${hardware_safety['read_transport_mode']}"
     use_fake_hardware="$(arg use_fake_hardware)"
-    arm_operating_mode="$(arg arm_operating_mode)"/>
+    arm_operating_mode="$(arg arm_operating_mode)"
+    torque_off_diagnostic_mode="$(arg torque_off_diagnostic_mode)"/>
 </robot>

File: om6dof_description/urdf/om6dof.urdf.xacro (robot description, xacro)
@@ -5,11 +5,33 @@
   <!-- Import Rviz colors -->
   <xacro:include filename="$(find om6dof_description)/urdf/materials.xacro" />
+  <!-- Pedestal from the ground/table plane to the bottom of the base servo. -->
+  <xacro:property name="base_height" value="0.020"/>
   <!-- World -->
   <link name="world">
   </link>
-  <!-- World fixed joint-->
+  <!-- A 20 mm support keeps the bottom of the link1/base servo above ground. -->
+  <link name="base_link">
+    <visual>
+      <!-- link1 footprint is approximately 46.5 x 28.5 mm; leave a 1.75 mm rim. -->
+      <origin xyz="0 0 ${base_height / 2.0}" rpy="0 0 0"/>
+      <geometry>
+        <box size="0.050 0.032 ${base_height}"/>
+      </geometry>
+      <material name="grey"/>
+    </visual>
+    <!-- Deliberately visual-only: the pedestal is fixed to the table plane,
+         so collision geometry here would permanently contact the table object
+         in MoveIt's planning scene. -->
+  </link>
+  <!-- World fixed joint: ground/table plane -> 20 mm pedestal. -->
   <joint name="world_fixed" type="fixed">
     <origin xyz="0 0 0" rpy="0 0 0"/>
     <parent link="world"/>
+    <child link="base_link"/>
+  </joint>
+  <!-- Pedestal top -> bottom of the base servo (link1). -->
+  <joint name="base_to_link1" type="fixed">
+    <origin xyz="0 0 ${base_height}" rpy="0 0 0"/>
+    <parent link="base_link"/>
     <child link="link1"/>
   </joint>
@@ -426,17 +448,8 @@
   <!-- end effector link -->
   <link name="end_effector_link">
-    <visual>
-      <origin xyz="0 0 0" rpy="0 0 0"/>
-      <geometry>
-        <box size="0.01 0.01 0.01" />
-      </geometry>
-      <material name="red"/>
-     </visual>
-    <collision>
-      <origin xyz="0 0 0" rpy="0 0 0"/>
-      <geometry>
-        <box size="0.01 0.01 0.01"/>
-      </geometry>
-    </collision>
+    <!-- Coordinate/inertial frame only. The former 10 mm red cube was a
+         debug glyph, not measured hardware, and made MoveIt collide against
+         a phantom object at the TCP. The finger links contain the physical
+         gripper visual/collision meshes. -->
     <inertial>
       <origin xyz="0.0 0.0 0.0" rpy="0 0 0"/>

Commit message: add f_gng

File: om6dof_bringup/urdf/om6dof.ros2_control.current.xacro (robot description, xacro)
@@ -100,4 +100,5 @@
       <joint name="${prefix}joint1">
         <command_interface name="position"/>
+        <command_interface name="position_offset"/>
         <command_interface name="effort"/>
         <state_interface name="position">
@@ -109,4 +110,5 @@
       <joint name="${prefix}joint2">
         <command_interface name="position"/>
+        <command_interface name="position_offset"/>
         <command_interface name="effort"/>
         <state_interface name="position">
@@ -118,4 +120,5 @@
       <joint name="${prefix}joint3">
         <command_interface name="position"/>
+        <command_interface name="position_offset"/>
         <command_interface name="effort"/>
         <state_interface name="position">
@@ -127,4 +130,5 @@
       <joint name="${prefix}joint4">
         <command_interface name="position"/>
+        <command_interface name="position_offset"/>
         <command_interface name="effort"/>
         <state_interface name="position">
@@ -136,4 +140,5 @@
       <joint name="${prefix}joint5">
         <command_interface name="position"/>
+        <command_interface name="position_offset"/>
         <command_interface name="effort"/>
         <state_interface name="position">
@@ -145,4 +150,5 @@
       <joint name="${prefix}joint6">
         <command_interface name="position"/>
+        <command_interface name="position_offset"/>
         <command_interface name="effort"/>
         <state_interface name="position">

File: om6dof_bringup/urdf/om6dof.ros2_control.xacro (robot description, xacro)
@@ -82,6 +82,14 @@
            which is a wrist singularity where Servo emergency-stops). On real
            hardware the dxl interface reads encoders and ignores these. -->
+      <!-- Two additive position command channels per arm joint.
+           `position`        : autonomous motion (MoveIt -> arm_controller).
+           `position_offset` : the human operator (om6dof_controller ->
+                               forward_offset_controller).
+           DynamixelHardware::write() sends their sum to the motor, so both
+           controllers stay active at once instead of taking turns over one
+           shared interface. The gripper keeps a single channel. -->
       <joint name="${prefix}joint1">
         <command_interface name="position"/>
+        <command_interface name="position_offset"/>
         <state_interface name="position">
           <param name="initial_value">0.0</param>
@@ -92,4 +100,5 @@
       <joint name="${prefix}joint2">
         <command_interface name="position"/>
+        <command_interface name="position_offset"/>
         <state_interface name="position">
           <param name="initial_value">-0.6806</param>
@@ -100,4 +109,5 @@
       <joint name="${prefix}joint3">
         <command_interface name="position"/>
+        <command_interface name="position_offset"/>
         <state_interface name="position">
           <param name="initial_value">1.3613</param>
@@ -108,4 +118,5 @@
       <joint name="${prefix}joint4">
         <command_interface name="position"/>
+        <command_interface name="position_offset"/>
         <state_interface name="position">
           <param name="initial_value">0.0</param>
@@ -116,4 +127,5 @@
       <joint name="${prefix}joint5">
         <command_interface name="position"/>
+        <command_interface name="position_offset"/>
         <state_interface name="position">
           <param name="initial_value">0.8901</param>
@@ -124,4 +136,5 @@
       <joint name="${prefix}joint6">
         <command_interface name="position"/>
+        <command_interface name="position_offset"/>
         <state_interface name="position">
           <param name="initial_value">0.0</param>

File: om6dof_bringup/urdf/om6dof.urdf.xacro (robot description, xacro)
@@ -19,5 +19,8 @@
   <xacro:property name="hardware_safety"
     value="${xacro.load_yaml('$(find om6dof_bringup)/config/hardware_safety.yaml')}"/>
-  <xacro:include filename="$(find om6dof_description)/urdf/om6dof.urdf.xacro"/>
+  <!-- The physical arm uses the v2 link3 mounting geometry. Keep the
+       robot_state_publisher/controller_manager model aligned with MoveIt,
+       direct pick, and Gemini pick. -->
+  <xacro:include filename="$(find om6dof_description)/urdf/om6dof_v2.urdf.xacro"/>
   <!-- Exactly one of these: both define om6dof_ros2_control, so including
        both would redefine the macro. -->

File: om6dof_description/urdf/om6dof_v2.urdf.xacro (robot description, xacro)
@@ -420,9 +420,27 @@
     </inertial>-->
   </link>
-  <!--  Gripper joint -->
+  <!-- TCP / end-effector control frame.  Keep this link between the wrist and
+       the gripper branches so MoveIt places its interactive marker at the TCP,
+       rather than at link7 (the wrist flange). -->
+  <joint name="end_effector_joint" type="fixed">
+    <origin xyz="0.0 0.0 0.115" rpy="0 0 0"/>
+    <parent link="link7"/>
+    <child link="end_effector_link"/>
+  </joint>
+  <link name="end_effector_link">
+    <!-- Coordinate/inertial frame only. The finger links contain the physical
+         gripper visual and collision meshes. -->
+    <inertial>
+      <origin xyz="0.0 0.0 0.0" rpy="0 0 0"/>
+      <mass value="0.001"/>
+      <inertia ixx="1.0e-06" ixy="0.0" ixz="0.0" iyy="1.0e-06" iyz="0.0" izz="1.0e-06" />
+    </inertial>
+  </link>
+  <!-- Gripper joints are expressed from the TCP.  -44.3 mm preserves their
+       original +70.7 mm pose relative to link7: 115.0 - 44.3 = 70.7 mm. -->
   <joint name="gripper_left_joint" type="prismatic">
-    <parent link="link7"/>
+    <parent link="end_effector_link"/>
     <child link="gripper_left_link"/>
-    <origin xyz="0.0 0.021 0.0707" rpy="0 0 0"/>
+    <origin xyz="0.0 0.021 -0.0443" rpy="0 0 0"/>
     <axis xyz="0 1 0"/>
     <limit velocity="4.8" effort="1000" lower="-0.011" upper="0.020" />
@@ -473,7 +491,7 @@
   <!--  Gripper joint sub -->
   <joint name="gripper_right_joint" type="prismatic">
-    <parent link="link7"/>
+    <parent link="end_effector_link"/>
     <child link="gripper_right_link"/>
-    <origin xyz="0.0 -0.021 0.0707" rpy="0 0 0"/>
+    <origin xyz="0.0 -0.021 -0.0443" rpy="0 0 0"/>
     <axis xyz="0 -1 0"/>
     <limit velocity="4.8" effort="1000" lower="-0.011" upper="0.020" />
@@ -481,22 +499,4 @@
     <mimic joint="gripper_left_joint" multiplier="1"/>
   </joint>
-  <!-- end effector joint -->
-  <joint name="end_effector_joint" type="fixed">
-    <origin xyz="0.0 0.0 0.115" rpy="0 0 0"/>
-    <parent link="link7"/>
-    <child link="end_effector_link"/>
-  </joint>
-  <!-- end effector link -->
-  <link name="end_effector_link">
-    <!-- Coordinate/inertial frame only. The former 10 mm red cube was a
-         debug glyph, not measured hardware, and made MoveIt collide against
-         a phantom object at the TCP. The finger links contain the physical
-         gripper visual/collision meshes. -->
-    <inertial>
-      <origin xyz="0.0 0.0 0.0" rpy="0 0 0"/>
-      <mass value="0.001"/>
-      <inertia ixx="1.0e-06" ixy="0.0" ixz="0.0" iyy="1.0e-06" iyz="0.0" izz="1.0e-06" />
-    </inertial>
-  </link>
   <!-- ==================== wrist payload (RealSense D435) ====================
        V2-only component masses and estimated CAD-frame centres of mass live
@@ -523,6 +523,6 @@
        The underside has a small slope; contact is aligned at the bolt axes.
        This is a mesh-based placement, not a measured optical calibration.
-       The d405_* optical transforms still need D435-specific calibration;
-       their old names are retained for consumers.
+       D435 optical frames below use CAD/nominal geometry, not the former
+       D405 extrinsic. Only the payload link/joint retain their legacy names.
   -->
   <xacro:property name="d435_mount_cad_x" value="0.051870518"/>
@@ -568,21 +568,55 @@
     </xacro:if>
   </link>
-  <!-- Legacy D405 optical transforms retained for existing consumers.
-       These values describe the former D405 assembly, not the D435 mesh above.
-       The original derivation remains in om6dof.urdf.xacro. Calibrate the D435
-       housing-to-optical transform before using these frames for perception.
+  <!-- D435 camera frames: measured CAD registration plus nominal manufacturer
+       lens offsets. These are NOT measured camera-to-arm hand-eye extrinsics.
+       The mounting pose, mesh, collision, and mass above are unchanged.
+       Keep physical/body and optical axes separate, and distinguish RGB from
+       depth: depth aligned to RGB is expressed in the colour optical frame.
+       Factory sensor-to-sensor extrinsics may differ from these nominal values.
+       See config/camera_d435.yaml for provenance and coordinate conventions.
   -->
-  <joint name="d405_link_joint" type="fixed">
-    <origin xyz="0.010093 0.047231 0.000046" rpy="-1.134465 1.570590 -1.570798"/>
+  <xacro:property name="d435_camera_cfg"
+                  value="${xacro.load_yaml('$(find om6dof_description)/config/camera_d435.yaml')}"/>
+  <xacro:property name="d435_camera" value="${d435_camera_cfg['camera']}"/>
+  <joint name="d435_bottom_screw_joint" type="fixed">
+    <origin xyz="${d435_camera['bottom_screw_cad_xyz'][0] - d435_mount_cad_x} ${d435_camera['bottom_screw_cad_xyz'][1] - d435_mount_cad_y} ${d435_camera['bottom_screw_cad_xyz'][2] - d435_mount_cad_z}"
+            rpy="${d435_camera['bottom_screw_rpy'][0]} ${d435_camera['bottom_screw_rpy'][1]} ${d435_camera['bottom_screw_rpy'][2]}"/>
     <parent link="d405_payload_link"/>
-    <child link="d405_link"/>
-  </joint>
-  <link name="d405_link"/>
-  <joint name="d405_depth_optical_joint" type="fixed">
-    <!-- Legacy D405 depth offset; not calibrated for the D435. -->
-    <origin xyz="0 0 -0.0037" rpy="0 0 ${pi}"/>
-    <parent link="d405_link"/>
-    <child link="d405_depth_optical_frame"/>
-  </joint>
-  <link name="d405_depth_optical_frame"/>
+    <child link="d435_bottom_screw_frame"/>
+  </joint>
+  <link name="d435_bottom_screw_frame"/>
+  <joint name="d435_link_joint" type="fixed">
+    <origin xyz="${d435_camera['depth_from_bottom_screw_xyz'][0]} ${d435_camera['depth_from_bottom_screw_xyz'][1]} ${d435_camera['depth_from_bottom_screw_xyz'][2]}"
+            rpy="0 0 0"/>
+    <parent link="d435_bottom_screw_frame"/>
+    <child link="d435_link"/>
+  </joint>
+  <link name="d435_link"/>
+  <joint name="d435_depth_joint" type="fixed">
+    <origin xyz="0 0 0" rpy="0 0 0"/>
+    <parent link="d435_link"/>
+    <child link="d435_depth_frame"/>
+  </joint>
+  <link name="d435_depth_frame"/>
+  <joint name="d435_depth_optical_joint" type="fixed">
+    <origin xyz="0 0 0"
+            rpy="${d435_camera['optical_rpy'][0]} ${d435_camera['optical_rpy'][1]} ${d435_camera['optical_rpy'][2]}"/>
+    <parent link="d435_depth_frame"/>
+    <child link="d435_depth_optical_frame"/>
+  </joint>
+  <link name="d435_depth_optical_frame"/>
+  <joint name="d435_color_joint" type="fixed">
+    <origin xyz="${d435_camera['color_from_depth_xyz'][0]} ${d435_camera['color_from_depth_xyz'][1]} ${d435_camera['color_from_depth_xyz'][2]}"
+            rpy="0 0 0"/>
+    <parent link="d435_link"/>
+    <child link="d435_color_frame"/>
+  </joint>
+  <link name="d435_color_frame"/>
+  <joint name="d435_color_optical_joint" type="fixed">
+    <origin xyz="0 0 0"
+            rpy="${d435_camera['optical_rpy'][0]} ${d435_camera['optical_rpy'][1]} ${d435_camera['optical_rpy'][2]}"/>
+    <parent link="d435_color_frame"/>
+    <child link="d435_color_optical_frame"/>
+  </joint>
+  <link name="d435_color_optical_frame"/>
 </robot>
