Commit message: fix urdf mass and CoM

File: om6dof_description/urdf/om6dof.urdf.xacro (robot description, xacro)
@@ -108,5 +108,17 @@
     </collision>
     <inertial>
-      <origin xyz="0 0 0" />
+      <!-- Centre of mass from the volume centroid of chain_link3.stl (61.15 cm^3),
+           taking the part as uniform density.
+           It replaces 0 0 0, which put this link's mass exactly on its own joint
+           axis. Across link3, link4, link5 and the two fingers that placeholder was
+           hiding about 0.0218 kg m of first moment, roughly 0.21 Nm of gravity
+           torque, near 18% of joint2 peak. That is the sort of error a fitted
+           scale factor cannot absorb, because it is distribution, not magnitude.
+           An estimate, not CAD. The implied density is well above plastic, so the
+           mass almost certainly includes a servo the mesh does not draw. Better
+           than the origin, worse than the real numbers link1, link2, link6 and
+           link7 carry. The inertia below is still the old placeholder; gravity
+           never reads it. -->
+      <origin xyz="0.0 4.5e-04 9.4132e-02" />
       <mass value="0.131" />
       <inertia ixx="0.1" ixy="0.0" ixz="0.0"
@@ -147,5 +159,17 @@
     </collision>
     <inertial>
-      <origin xyz="0 0 0" />
+      <!-- Centre of mass from the volume centroid of chain_link4.stl (47.44 cm^3),
+           taking the part as uniform density.
+           It replaces 0 0 0, which put this link's mass exactly on its own joint
+           axis. Across link3, link4, link5 and the two fingers that placeholder was
+           hiding about 0.0218 kg m of first moment, roughly 0.21 Nm of gravity
+           torque, near 18% of joint2 peak. That is the sort of error a fitted
+           scale factor cannot absorb, because it is distribution, not magnitude.
+           An estimate, not CAD. The implied density is well above plastic, so the
+           mass almost certainly includes a servo the mesh does not draw. Better
+           than the origin, worse than the real numbers link1, link2, link6 and
+           link7 carry. The inertia below is still the old placeholder; gravity
+           never reads it. -->
+      <origin xyz="-1.1470e-02 1.0e-05 4.3690e-02" />
       <mass value="0.098" />
       <inertia ixx="0.1" ixy="0.0" ixz="0.0"
@@ -186,5 +210,17 @@
     </collision>
     <inertial>
-      <origin xyz="0 0 0" />
+      <!-- Centre of mass from the volume centroid of chain_link5.stl (45.10 cm^3),
+           taking the part as uniform density.
+           It replaces 0 0 0, which put this link's mass exactly on its own joint
+           axis. Across link3, link4, link5 and the two fingers that placeholder was
+           hiding about 0.0218 kg m of first moment, roughly 0.21 Nm of gravity
+           torque, near 18% of joint2 peak. That is the sort of error a fitted
+           scale factor cannot absorb, because it is distribution, not magnitude.
+           An estimate, not CAD. The implied density is well above plastic, so the
+           mass almost certainly includes a servo the mesh does not draw. Better
+           than the origin, worse than the real numbers link1, link2, link6 and
+           link7 carry. The inertia below is still the old placeholder; gravity
+           never reads it. -->
+      <origin xyz="0.0 6.1e-04 4.6800e-02" />
       <mass value="0.098" />
       <inertia ixx="0.1" ixy="0.0" ixz="0.0"
@@ -225,6 +261,16 @@
     </collision>
      <inertial>
-      <origin xyz="4.4206755e-02 3.6839985e-07 8.9142216e-03" />
-      <mass value="1.4327573e-01" />
+      <!-- This link carried link7's inertial block verbatim: same mass, same centre
+           of mass, same tensor, for a different part. No permutation or sign flip of
+           that centre of mass lands inside chain_link6.stl, whose largest half extent
+           is 28 mm against the 44.2 mm written there, so it was never link6's number
+           to begin with.
+           Replaced with this mesh's own volume centroid, on the same uniform-density
+           assumption used on link3, link4 and link5.
+           The MASS is left alone but is not trusted either: 143 g against 4.38 cm^3
+           of mesh is 32.7 g/cm^3, denser than lead. Either the servo is not drawn
+           here, or this was copied from link7 too. Real CAD is what settles it. -->
+      <origin xyz="0.0 0.0 2.0370e-02" />
+      <mass value="0.04605" />
       <inertia ixx="8.0870749e-05" ixy="0.0" ixz="-1.0157896e-06"
                iyy="7.5980465e-05" iyz="0.0"
@@ -257,6 +303,11 @@
     </collision>
      <inertial>
-      <origin xyz="4.4206755e-02 3.6839985e-07 8.9142216e-03" />
-      <mass value="1.4327573e-01" />
+      <!-- x and z were swapped here. Ray-cast against chain_link7.stl: the value as
+           written, 44.2 mm along +X, falls outside the body entirely, and of every
+           permutation and sign flip of the three numbers only those putting 44.2 on
+           Z land inside it. Keeping y as the near-zero component is the single-swap
+           reading and the one consistent with a symmetric part. -->
+      <origin xyz="-8.9142216e-03 3.6839985e-07 ${0.5*4.4206755e-02}" />
+      <mass value="0.22527573" />
       <inertia ixx="8.0870749e-05" ixy="0.0" ixz="-1.0157896e-06"
                iyy="7.5980465e-05" iyz="0.0"
@@ -280,5 +331,17 @@
     </collision>
     <inertial>
-      <origin xyz="0 0 0" />
+      <!-- Centre of mass from the volume centroid of the gripper mesh (27.19 cm^3),
+           taking the part as uniform density.
+           It replaces 0 0 0, which put this link's mass exactly on its own joint
+           axis. Across link3, link4, link5 and the two fingers that placeholder was
+           hiding about 0.0218 kg m of first moment, roughly 0.21 Nm of gravity
+           torque, near 18% of joint2 peak. That is the sort of error a fitted
+           scale factor cannot absorb, because it is distribution, not magnitude.
+           An estimate, not CAD. The implied density is well above plastic, so the
+           mass almost certainly includes a servo the mesh does not draw. Better
+           than the origin, worse than the real numbers link1, link2, link6 and
+           link7 carry. The inertia below is still the old placeholder; gravity
+           never reads it. -->
+      <origin xyz="0.0 9.3200e-03 1.0080e-02" />
       <mass value="0.017" />
       <inertia ixx="1.0e-03" ixy="0.0" ixz="0.0"
@@ -319,5 +382,17 @@
     </collision>
     <inertial>
-      <origin xyz="0 0 0" />
+      <!-- Centre of mass from the volume centroid of the gripper mesh (27.22 cm^3),
+           taking the part as uniform density.
+           It replaces 0 0 0, which put this link's mass exactly on its own joint
+           axis. Across link3, link4, link5 and the two fingers that placeholder was
+           hiding about 0.0218 kg m of first moment, roughly 0.21 Nm of gravity
+           torque, near 18% of joint2 peak. That is the sort of error a fitted
+           scale factor cannot absorb, because it is distribution, not magnitude.
+           An estimate, not CAD. The implied density is well above plastic, so the
+           mass almost certainly includes a servo the mesh does not draw. Better
+           than the origin, worse than the real numbers link1, link2, link6 and
+           link7 carry. The inertia below is still the old placeholder; gravity
+           never reads it. -->
+      <origin xyz="0.0 -9.3200e-03 1.0070e-02" />
       <mass value="0.017" />
       <inertia ixx="1.0e-03" ixy="0.0" ixz="0.0"

Commit message: add gravity compensation

File: om6dof_description/urdf/om6dof.urdf.xacro (robot description, xacro)
@@ -510,3 +510,76 @@
     </xacro:if>
   </link>
+  <!-- ============ D405 optical frame: d405_link, d405_depth_optical_frame ============
+       Everything above (d405_payload_link) places the ALOHA bracket + camera as one fused
+       STL. This section locates two more frames INSIDE that assembly: the camera's own body
+       frame (d405_link) and the depth optical frame tf2/RViz/librealsense-adjacent code
+       expects (z forward into the scene, x right, y down; REP 103 optical convention).
+       METHOD, splitting the fused mesh:
+       d405_wrist_cam.stl decomposes into exactly two disjoint shells by connected components
+       (union-find over shared vertices, since the bracket and camera don't touch): 19.32 cm^3
+       (the bracket) and 38.73 cm^3. The second is byte-for-byte the same geometry as
+       meshes/d405.stl: same 4630 triangles, same 38.73 cm^3, same triangle order, so that
+       file is the bare D405 camera body on its own, and the assembly contains one unmodified,
+       rigidly-placed copy of it. Kabsch/SVD alignment of that shell's 13890 vertices against
+       d405.stl's own vertices (both already in matching order, so vertex i corresponds to
+       vertex i, no nearest-neighbour search needed) recovers the placement to sub-micron
+       residual (max 5.9e-6 mm over 13890 points): not a noisy fit, effectively reading the
+       exact rigid transform back out of the file. A point given in d405.stl's own frame (mm)
+       maps through a fitted rotation R and translation t to the same point in the raw
+       d405_wrist_cam.stl frame (mm): the same frame the visual mesh origin above is stated in.
+       Composing t with that visual origin's shift (+19.1,-27.2,-75.5 mm, the same constant
+       used above) gives d405_link's origin in the d405_payload_link frame; R (pure rotation,
+       untouched by translation) gives its orientation directly. (Script: SVD/Kabsch alignment
+       of the two meshes, run once during this integration; not checked in.)
+       ORIENTATION SIGN, which way d405_link's +Z points:
+       d405.stl's own frame does not self-label which flat 42x42 end is the lens side and
+       which is the connector side: both end caps are otherwise plain, and the only
+       asymmetric feature found (two holes 18 mm apart, symmetric about the centerline, at
+       one extreme) could honestly be either the two imager lenses (18 mm matches the D405
+       baseline, Table 3-49 of the Intel D400 datasheet, doc 337029-017) or the two M3x0.5
+       mounting inserts on the back panel (Figure 4-9, same document). Rather than guess, the
+       sign was fixed by the one fact that has to hold regardless of mesh cosmetics: a wrist
+       camera must look away from the arm, roughly toward end_effector_link (link7 +Z), not
+       back into it. Of the two candidate directions +/-Z of d405.stl's own frame, local +Z
+       lands 25.0 deg off link7's +Z once carried through this whole chain; the other
+       candidate lands 155.0 deg off, looking back into the arm. So local +Z of d405.stl is
+       "forward" (into the scene), which also fixes local Z=0 as the front glass plane (the
+       housing only occupies local z in [-23, 0] mm).
+       This is the same kind of 180 degree call the bracket rotation above settled with a
+       photograph; no such photograph of the assembled camera exists here, so this is the next
+       best evidence available. If the world-frame point cloud is later seen to rotate or
+       drift as the wrist reorients, rather than sitting still (which is the actual M2
+       acceptance test), suspect this sign first.
+       DEPTH ORIGIN, where along that axis:
+       Table 4-16 (Figure 4-4) gives the D405 "Depth Start Point" as 3.7 mm behind the front
+       cover glass, i.e. 3.7 mm in local -Z from d405_link's origin. Table 4-21 places the
+       left imager 9 mm off the housing centerline (half of the 18 mm baseline), but which
+       side is "left" is not recoverable from this mesh (both end faces are bilaterally
+       symmetric in it; unlike the bracket rotation there is no photo of the assembled camera
+       to check against). That 9 mm is left off (optical frame kept on the centerline) rather
+       than guessing its sign: it only shifts the drawn TF pose in RViz, never the
+       reconstructed point cloud, because the perception node deprojects with librealsense's
+       own live intrinsics (fx, fy, ppx, ppy read from the camera at runtime), not this static
+       offset.
+       d405_depth_optical_frame's rotation relative to d405_link is left as identity: baseline
+       (d405.stl local X) lands within 0.012 deg of link7's own +Y axis, and forward (local Z)
+       within 25 deg of link7's +Z, exactly what X-right/Y-down/Z-forward should look like if
+       d405.stl's mesh axes were already authored in that convention, which is plausible for a
+       mesh sourced for URDF/ROS use. Like the 9 mm above, this is not verified against the
+       real hardware's markings.
+  -->
+  <joint name="d405_link_joint" type="fixed">
+    <origin xyz="0.010093 0.047231 0.000046" rpy="-1.134465 1.570590 -1.570798"/>
+    <parent link="d405_payload_link"/>
+    <child link="d405_link"/>
+  </joint>
+  <link name="d405_link"/>
+  <joint name="d405_depth_optical_joint" type="fixed">
+    <!-- -0.0037 m: Table 4-16 "Depth Start Point" for D405, 3.7 mm behind the front cover
+         glass (local -Z, back toward the sensor); see the derivation above. -->
+    <origin xyz="0 0 -0.0037" rpy="0 0 0"/>
+    <parent link="d405_link"/>
+    <child link="d405_depth_optical_frame"/>
+  </joint>
+  <link name="d405_depth_optical_frame"/>
 </robot>

Commit message: update controller

File: om6dof_description/urdf/om6dof.urdf.xacro (robot description, xacro)
@@ -72,5 +72,5 @@
     <origin xyz="0.012 0.0 0.017" rpy="0 0 0"/>
     <axis xyz="0 0 1"/>
-    <limit velocity="4.8" effort="1" lower="${-pi*0.9}" upper="${pi*0.9}" />
+    <limit velocity="4.8" effort="1" lower="${-pi*0.5}" upper="${pi*0.5}" />
     <dynamics damping="0.1"/>
   </joint>
@@ -162,5 +162,5 @@
     <origin xyz="0.0 0 0.124" rpy="0 0 0"/>
     <axis xyz="0 1 0"/>
-    <limit velocity="4.8" effort="1" lower="${-pi*0.60}" upper="${pi*0.68}" />
+    <limit velocity="4.8" effort="1" lower="${-pi*0.5}" upper="${pi*0.68}" />
     <dynamics damping="0.1"/>
   </joint>
@@ -213,5 +213,5 @@
     <origin xyz="0.0 0.0 0.045" rpy="0 0 0"/>
     <axis xyz="0 0 1"/>
-    <limit velocity="4.8" effort="1" lower="${-pi*0.9}" upper="${pi*0.9}" />
+    <limit velocity="4.8" effort="1" lower="${-pi*0.4}" upper="${pi*0.4}" />
     <dynamics damping="0.1"/>
   </joint>
@@ -264,5 +264,5 @@
     <origin xyz="0.0 0.0 0.0595" rpy="0 0 0"/>
     <axis xyz="0 1 0"/>
-    <limit velocity="4.8" effort="1" lower="${-pi*0.63}" upper="${pi*0.67}" />
+    <limit velocity="4.8" effort="1" lower="${-pi*0.5}" upper="${pi*0.67}" />
     <dynamics damping="0.1"/>
   </joint>
@@ -306,5 +306,5 @@
     <origin xyz="0.0 0.0 0.0475" rpy="0 0 0"/>
     <axis xyz="0 0 1"/>
-    <limit velocity="4.8" effort="1" lower="${-pi*0.9}" upper="${pi*0.9}" />
+    <limit velocity="4.8" effort="1" lower="${-pi*0.5}" upper="${pi*0.5}" />
     <dynamics damping="0.1"/>
   </joint>
